File: electronics/Fenix.kicad_pcb (KiCad board)
At the start: 2 copper layers, 126 x 54 mm, 8 parts

Commit message: Update Symbol/Footprint link & Remove GPS board
Parts:
- removed U3: ~, Parts:LORA32_V4
- removed U5: ~, Parts:Adafruit_GPSFeather
- added J1: PWR, TerminalBlock:TerminalBlock_MaiXu_MX126-5.0-02P_1x02_P5.00mm, F.Cu at (183.0, 71.9)
- added J2: RELAY_CTRL, TerminalBlock:TerminalBlock_MaiXu_MX126-5.0-02P_1x02_P5.00mm, F.Cu at (183.0, 82.0)
- added LoRa32_V1: ~, Parts:LORA32_V4, F.Cu at (162.4, 78.0)
- renumbered U1 to Gyro1, U2 to Servo_Controller1, U4 to uSD1
Connections:
- TEMP_EXT1 pad 1: (no net) -> +3V3
- TEMP_EXT1 pad 2: (no net) -> GND
- TEMP_EXT1 pad 3: (no net) -> /I2C_CLK
- TEMP_EXT1 pad 4: (no net) -> /I2C_DATA
- TEMP_INT1 pad 1: (no net) -> +3V3
- TEMP_INT1 pad 2: (no net) -> GND
- TEMP_INT1 pad 3: (no net) -> /I2C_CLK
- TEMP_INT1 pad 4: (no net) -> /I2C_DATA

Commit message: Organize nets/symbols
Parts:
- removed J1: PWR, TerminalBlock:TerminalBlock_MaiXu_MX126-5.0-02P_1x02_P5.00mm
- added J1_5VIN1: PWR, TerminalBlock:TerminalBlock_MaiXu_MX126-5.0-02P_1x02_P5.00mm, F.Cu at (183.0, 72.0)
Connections:
- Gyro1 pad 1: unconnected-(Gyro1-VIN-Pad1) -> +5V
- Gyro1 pad 2: +3V3 -> unconnected-(Gyro1-3vo-Pad2)
- Gyro1 pad 4: unconnected-(Gyro1-SDA-Pad4) -> /I2C_DATA
- Gyro1 pad 5: unconnected-(Gyro1-SCL-Pad5) -> /I2C_CLK
- Gyro1 pad 7: unconnected-(Gyro1-ADR-Pad7) -> Net-(Gyro1-ADR)
- Servo_Controller1 pad 10: unconnected-(Servo_Controller1-SCL-Pad10) -> /I2C_CLK
- Servo_Controller1 pad 9: unconnected-(Servo_Controller1-SDA-Pad9) -> /I2C_DATA
Changed lines of the file:
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@@
 			(layers "*.Cu" "*.Mask")
 			(remove_unused_layers no)
-			(net "unconnected-(Gyro1-VIN-Pad1)")
+			(net "+5V")
 			(pinfunction "VIN_1")
 			(pintype "power_in")
@@
 			(layers "*.Cu" "*.Mask")
 			(remove_unused_layers no)
-			(net "+3V3")
+			(net "unconnected-(Gyro1-3vo-Pad2)")
 			(pinfunction "3vo_2")
 			(pintype "power_out")
@@
 			(layers "*.Cu" "*.Mask")
 			(remove_unused_layers no)
-			(net "unconnected-(Gyro1-SDA-Pad4)")
+			(net "/I2C_DATA")
 			(pinfunction "SDA_4")
 			(pintype "bidirectional")
@@
 			(layers "*.Cu" "*.Mask")
 			(remove_unused_layers no)
-			(net "unconnected-(Gyro1-SCL-Pad5)")
+			(net "/I2C_CLK")
 			(pinfunction "SCL_5")
 			(pintype "input")
@@
 			(layers "*.Cu" "*.Mask")
 			(remove_unused_layers no)
-			(net "unconnected-(Gyro1-ADR-Pad7)")
+			(net "Net-(Gyro1-ADR)")
 			(pinfunction "ADR_7")
 			(pintype "input")
@@
 			(layers "*.Cu" "*.Mask")
 			(remove_unused_layers no)
-			(net "unconnected-(Servo_Controller1-SDA-Pad9)")
+			(net "/I2C_DATA")
 			(pinfunction "SDA_9")
 			(pintype "bidirectional")
@@
 			(layers "*.Cu" "*.Mask")
 			(remove_unused_layers no)
-			(net "unconnected-(Servo_Controller1-SCL-Pad10)")
+			(net "/I2C_CLK")
 			(pinfunction "SCL_10")
 			(pintype "input")
@@
 	(footprint "TerminalBlock:TerminalBlock_MaiXu_MX126-5.0-02P_1x02_P5.00mm"
 		(layer "F.Cu")
-		(at 183 71.885)
+		(at 183 72)
 		(descr "terminal block MaiXu MX126-5.0-02P, 2 pins, pitch 5mm, size 10.5x7.8mm, drill diameter 1.3mm, pad diameter 2.8mm, https://www.lcsc.com/datasheet/lcsc_datasheet_2309150913_MAX-MX126-5-0-03P-GN01-Cu-S-A_C5188435.pdf, script-generated using https://gitlab.com/kicad/libraries/kicad-footprint-generator/-/tree/master/scripts/TerminalBlock_MaiXu")
 		(tags "THT terminal block MaiXu MX126-5.0-02P pitch 5mm size 10.5x7.8mm drill 1.3mm pad 2.8mm")
-		(property "Reference" "J1"
+		(property "Reference" "J1_5VIN1"
 			(at 2.25 -5.12 0)
 			(layer "F.SilkS")
@@
 			(remove_unused_layers no)
 			(roundrect_rratio 0.089286)
-			(net "unconnected-(J1-Pin_1-Pad1)")
+			(net "+5V")
 			(pinfunction "Pin_1_1")
 			(pintype "passive")
@@
 			(layers "*.Cu" "*.Mask")
 			(remove_unused_layers no)
-			(net "unconnected-(J1-Pin_2-Pad2)")
+			(net "GND")
 			(pinfunction "Pin_2_2")
 			(pintype "passive")

Commit message: Hardware Night: Finish schematic and PCB routing for known parts
Parts:
- added J3_ADR1: Conn_01x02_Pin, Connector_PinHeader_2.54mm:PinHeader_1x02_P2.54mm_Vertical, F.Cu at (115.7, 77.0)
- added J4_SRV_EN1: Conn_01x02_Pin, Connector_PinHeader_2.54mm:PinHeader_1x02_P2.54mm_Vertical, F.Cu at (104.7, 57.5)
- moved TEMP_EXT1 85.7 mm to (104.9, 112.5), turned to 0 degrees
- moved uSD1 83.5 mm to (112.7, 72.2), turned to 90 degrees
- moved G*** 53.3 mm to (125.5, 111.0)
- moved J1_5VIN1 45.0 mm to (162.2, 112.0)
- moved TEMP_INT1 36.8 mm to (111.1, 77.0)
- moved J2 31.0 mm to (209.2, 98.5)
- moved Gyro1 26.6 mm to (111.0, 93.0)
- moved Servo_Controller1 25.7 mm to (87.0, 85.5), turned to -90 degrees
- moved LoRa32_V1 23.8 mm to (144.6, 93.9), turned to 180 degrees
Connections:
- Gyro1 pad 6: unconnected-(Gyro1-RST-Pad6) -> /GYRO_RST
- LoRa32_V1 pad 09: unconnected-(LoRa32_V1-G36-Pad09) -> /SPI_CLK
- LoRa32_V1 pad 10: unconnected-(LoRa32_V1-G35-Pad10) -> /SPI_PICO
- LoRa32_V1 pad 11: unconnected-(LoRa32_V1-G34-Pad11) -> /SPI_CS_SD
- LoRa32_V1 pad 13: unconnected-(LoRa32_V1-G47-Pad13) -> /I2C_CLK
- LoRa32_V1 pad 14: unconnected-(LoRa32_V1-G48-Pad14) -> /I2C_DATA
- LoRa32_V1 pad 15: unconnected-(LoRa32_V1-G26-Pad15) -> /GYRO_RST
- LoRa32_V1 pad 33: unconnected-(LoRa32_V1-G37-Pad33) -> /SPI_POCI
- Servo_Controller1 pad 11: unconnected-(Servo_Controller1-OE-Pad11) -> Net-(J4_SRV_EN1-Pin_1)
- Servo_Controller1 pad 2: unconnected-(Servo_Controller1-OE-Pad2) -> /SERVO_EN
- Servo_Controller1 pad 3: unconnected-(Servo_Controller1-SCL-Pad3) -> /I2C_CLK
- Servo_Controller1 pad 4: unconnected-(Servo_Controller1-SDA-Pad4) -> /I2C_DATA
- uSD1 pad 2: unconnected-(uSD1-CS-Pad2) -> /SPI_CS_SD
- uSD1 pad 3: unconnected-(uSD1-PICO-Pad3) -> /SPI_PICO
- uSD1 pad 4: unconnected-(uSD1-CLK-Pad4) -> /SPI_CLK
- uSD1 pad 5: unconnected-(uSD1-POCI-Pad5) -> /SPI_POCI
Routing:
- net GND: track 0.00 -> 190.0 mm
- net /I2C_CLK: track 0.00 -> 187.6 mm, vias 0 -> 3
- net /I2C_DATA: track 0.00 -> 187.2 mm
- net +5V: track 0.00 -> 167.2 mm, vias 0 -> 1
- net +3V3: track 0.00 -> 165.4 mm, vias 0 -> 1
- net /GYRO_RST: track 0.00 -> 71.5 mm, vias 0 -> 1
- net Net-(J4_SRV_EN1-Pin_1): track 0.00 -> 62.6 mm
- net /SPI_CS_SD: track 0.00 -> 53.3 mm, vias 0 -> 1
- net /SPI_CLK: track 0.00 -> 52.5 mm, vias 0 -> 1
- net /SPI_PICO: track 0.00 -> 50.6 mm, vias 0 -> 1
- net /SPI_POCI: track 0.00 -> 39.2 mm
- net Net-(Gyro1-ADR): track 0.00 -> 22.1 mm
Other:
- board size 126 x 54 mm -> 116.5 x 64 mm
- board text added: "2.4G WiFi"
- board text added: "5v Out"
- board text added: "From by Andrew Young, Disaster Fonts. & downloaded from https://www.dafont.com/lazenby-computer.font"
- board text added: "Gyro"
- board text added: "HEATER"
- board text added: "LORA32 V4"
- board text added: "SD CARD"
- board text added: "Servo Controller"
- board text added: "TEMP INT"
- board text added: "Temp Ext"

Commit message: Some PCB layout, will need to redo 3.5mm jack footprint
Parts:
- added A1: RaspberryPi_Pico, Module:RaspberryPi_Pico_Common_Unspecified, F.Cu at (174.5, 80.5)
- added C1: 100nF, Capacitor_THT:C_Disc_D4.3mm_W1.9mm_P5.00mm, F.Cu at (188.5, 101.0)
- added C2: 4.7nF, Capacitor_THT:C_Disc_D4.3mm_W1.9mm_P5.00mm, F.Cu at (197.0, 113.0)
- added D1: 1N5817, Diode_THT:D_DO-41_SOD81_P10.16mm_Horizontal, F.Cu at (159.5, 81.4)
- added D2: 1N5817, Diode_THT:D_DO-41_SOD81_P10.16mm_Horizontal, F.Cu at (159.5, 107.6)
- added J1: Radio 3.5mm, Parts:TRS_3.5mm, F.Cu at (209.8, 74.3)
- added J3: Radio 2.5mm, Parts:TRS_2.5mm, F.Cu at (194.0, 88.5)
- added J4_LORA_PWR1: Conn_01x02_Pin, Connector_PinHeader_2.54mm:PinHeader_1x02_P2.54mm_Vertical, F.Cu at (160.0, 111.0)
- added J_PWR1: Conn_01x03_Pin, Connector_PinHeader_1.00mm:PinHeader_1x03_P1.00mm_Horizontal, F.Cu at (209.6, 125.5)
- added Q1: BC548, Package_TO_SOT_THT:TO-92_Inline, F.Cu at (193.5, 97.9)
- added R1: 4k7, Resistor_THT:R_Axial_DIN0207_L6.3mm_D2.5mm_P7.62mm_Horizontal, F.Cu at (188.5, 104.5)
- added R2: 4k7, Resistor_THT:R_Axial_DIN0207_L6.3mm_D2.5mm_P7.62mm_Horizontal, F.Cu at (194.3, 109.0)
- added R3: 1k, Resistor_THT:R_Axial_DIN0207_L6.3mm_D2.5mm_P7.62mm_Horizontal, F.Cu at (183.6, 109.0)
- moved J2 31.3 mm to (221.0, 127.5)
- moved J1_5VIN1 3.25 mm to (165.5, 112.0)
Connections:
- LoRa32_V1 pad 02: +5V -> Net-(J4_LORA_PWR1-Pin_2)
- LoRa32_V1 pad 19: unconnected-(LoRa32_V1-G07-Pad19) -> /APRS_TX
- LoRa32_V1 pad 20: unconnected-(LoRa32_V1-G06-Pad20) -> /APRS_RX
Routing:
- net GND: track 190.0 -> 0.00 mm
- net /I2C_CLK: track 187.6 -> 0.00 mm, vias 3 -> 0
- net /I2C_DATA: track 187.2 -> 0.00 mm
- net +5V: track 167.2 -> 0.00 mm, vias 1 -> 0
- net +3V3: track 165.4 -> 0.00 mm, vias 1 -> 0
- net /GYRO_RST: track 71.5 -> 0.00 mm, vias 1 -> 0
- net Net-(J4_SRV_EN1-Pin_1): track 62.6 -> 0.00 mm
- net /SPI_CS_SD: track 53.3 -> 0.00 mm, vias 1 -> 0
- net /SPI_CLK: track 52.5 -> 0.00 mm, vias 1 -> 0
- net /SPI_PICO: track 50.6 -> 0.00 mm, vias 1 -> 0
- net /SPI_POCI: track 39.2 -> 0.00 mm
- net Net-(Gyro1-ADR): track 22.1 -> 0.00 mm
Other:
- board size 116.5 x 64 mm -> 126 x 64 mm
- board text added: "5v"
- board text removed: "2.4G WiFi"
- board text removed: "5v Out"

Commit message: Pre-Routing Board Layout
Parts:
- removed J1_5VIN1: PWR, TerminalBlock:TerminalBlock_MaiXu_MX126-5.0-02P_1x02_P5.00mm
- removed J_PWR1: Conn_01x03_Pin, Connector_PinHeader_1.00mm:PinHeader_1x03_P1.00mm_Horizontal
- added J4: PWR_MON, Connector_PinHeader_2.54mm:PinHeader_2x02_P2.54mm_Vertical, F.Cu at (183.7, 109.2)
- added J5: PWR_IN, TerminalBlock_Altech:Altech_AK100_1x02_P5.00mm, F.Cu at (192.0, 112.4)
- J2: value RELAY_CTRL -> Relay_Control; footprint TerminalBlock:TerminalBlock_MaiXu_MX126-5.0-02P_1x02_P5.00mm -> Connector_Phoenix_MSTB:PhoenixContact_MSTBVA_2,5_3-G_1x03_P5.00mm_Vertical
- moved J2 56.0 mm to (167.0, 112.5)
- moved J4_LORA_PWR1 25.9 mm to (134.2, 113.5), turned to 90 degrees
- moved J1 18.7 mm to (195.0, 63.0)
- moved C2 16.2 mm to (199.5, 97.0)
- moved R3 14.9 mm to (195.8, 100.5)
- moved J3 13.1 mm to (198.0, 76.0)
- moved R2 12.6 mm to (195.8, 96.5)
- moved C1 12.5 mm to (188.5, 88.5)
- moved Q1 12.5 mm to (193.5, 85.4)
- moved R1 12.0 mm to (188.2, 92.5)
- moved LoRa32_V1 6.47 mm to (144.1, 87.5)
- moved J4_SRV_EN1 2.06 mm to (104.2, 59.5)
- moved A1 2.00 mm to (174.5, 78.5)
- moved TEMP_EXT1 1.98 mm to (104.9, 110.5)
Connections:
- J2 pad 1: unconnected-(J2-Pin_1-Pad1) -> GND
- J2 pad 2: unconnected-(J2-Pin_2-Pad2) -> /RELAY_EN
- LoRa32_V1 pad 23: unconnected-(LoRa32_V1-G03-Pad23) -> /RELAY_EN
Other:
- board size 126 x 64 mm -> 130.5 x 64 mm
- board text added: "5-30V"
- board text added: "APRS"
- board text added: "GYRO ADDR"
- board text added: "HEAT"
- board text added: "LORA EN"
- board text added: "MON"
- board text added: "Pi PICO"
- board text added: "SERVO EN"
- board text added: "WE ARE THE MUSIC MAKERS AND WE ARE THE DREAMERS OF DREAMS"
- board text removed: "5v"
- board text removed: "HEATER"

Commit message: Completed PCB Design
Routing:
- net GND: track 0.00 -> 393.0 mm, vias 0 -> 7
- net +3V3: track 0.00 -> 256.9 mm
- net +5V: track 0.00 -> 177.5 mm, vias 0 -> 2
- net /I2C_DATA: track 0.00 -> 171.2 mm, vias 0 -> 1
- net /I2C_CLK: track 0.00 -> 165.5 mm, vias 0 -> 2
- net Net-(A1-VSYS): track 0.00 -> 112.5 mm
- net Net-(A1-GPIO8): track 0.00 -> 75.5 mm, vias 0 -> 2
- net /RELAY_EN: track 0.00 -> 74.2 mm, vias 0 -> 1
- net /GYRO_RST: track 0.00 -> 74.2 mm, vias 0 -> 1
- net Net-(J4_SRV_EN1-Pin_1): track 0.00 -> 60.4 mm
- net Net-(A1-GPIO9): track 0.00 -> 53.7 mm, vias 0 -> 1
- net /SPI_CS_SD: track 0.00 -> 50.6 mm, vias 0 -> 1
- net Net-(C2-Pad1): track 0.00 -> 49.7 mm
- net /SPI_PICO: track 0.00 -> 46.9 mm, vias 0 -> 1
- net /SPI_CLK: track 0.00 -> 45.4 mm, vias 0 -> 1
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- added copper zone on B.Cu, net GND
- added copper zone on F.Cu, net GND
